File: electrical/metro.kicad_pcb (KiCad board)
At the start: 4 copper layers, 28 x 30 mm, 37 parts, among them J1 Conn_01x02, J2 Conn_01x02, J3 Conn_01x02, Q1 AO3401A, U1 MCP73831T-2ACI/OT, U2 ATTINY1616-MN, U3 DRV2605LDGS, U4 XC6206P332MR-G

Commit message: Routing done
Parts:
- removed TP1: UPDI, TestPoint:TestPoint_THTPad_D1.0mm_Drill0.5mm
- added J4: Conn_01x03, Connector_Wire:SolderWire-0.1sqmm_1x03_P3.6mm_D0.4mm_OD1mm, F.Cu at (62.0, 90.6)
- moved D6 17.0 mm to (42.0, 73.0), turned to 90 degrees
- moved C6 16.0 mm to (52.8, 79.6), turned to 180 degrees
- moved C4 14.3 mm to (54.3, 86.2)
- moved U3 14.3 mm to (52.3, 83.4)
- moved C5 14.3 mm to (55.4, 86.2)
- moved R7 13.7 mm to (44.0, 71.7), turned to -90 degrees
- moved R8 7.86 mm to (54.7, 84.2), turned to -90 degrees
- moved R9 6.12 mm to (54.7, 82.2), turned to 90 degrees
- moved C3 3.02 mm to (62.4, 82.8)
- moved U2 3.02 mm to (59.7, 83.0)
- moved C7 2.83 mm to (46.5, 80.3)
- moved D7 1.60 mm to (43.0, 81.5)
- moved R10 1.60 mm to (42.4, 79.9)
- moved U4 1.60 mm to (46.5, 83.4)
- moved Q1 1.59 mm to (42.7, 84.2)
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Connections:
- D6 pad A: +VBUS -> Net-(D6-PadA)
- D6 pad C: Net-(D6-PadC) -> /LIPO STAT
- R7 pad 1: /LIPO STAT -> Net-(D6-PadA)
- R7 pad 2: Net-(D6-PadC) -> +VBUS
- U2 pad 1: /SW3 -> /SW2
- U2 pad 12: /SW2 -> /SW3
Routing:
- net +VBUS: track 0.00 -> 29.0 mm, vias 0 -> 2
- net GND: track 3.64 -> 24.7 mm, vias 3 -> 17
- net /SW1: track 0.00 -> 17.9 mm
- net /MOTOR-: track 0.00 -> 17.8 mm
- net /SW3: track 0.00 -> 16.8 mm, vias 0 -> 2
- net /LED1: track 0.00 -> 16.4 mm
- net /LIPO STAT: track 0.00 -> 15.6 mm, vias 0 -> 2
- net +BATT: track 0.00 -> 14.0 mm, vias 0 -> 1
- net +3V3: track 8.74 -> 22.1 mm, vias 3 -> 12
- net /LED2: track 0.00 -> 13.0 mm
- net /MOTOR+: track 0.00 -> 12.3 mm
- net /SW2: track 0.00 -> 9.95 mm
- net /LED3: track 0.00 -> 9.75 mm
- net /LED4: track 0.00 -> 7.36 mm
- net /LED5: track 0.00 -> 7.25 mm
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Other:
- outline, holes or cut-outs redrawn
- board text added: "3V3"
- board text added: "UPDI"

Commit message: shift things away from edges, remove dead tracks
Parts:
- moved U1 1.67 mm to (42.9, 89.4)
- moved C1 1.62 mm to (42.3, 91.7), turned to 0 degrees
- moved C2 1.43 mm to (44.5, 91.7), turned to 0 degrees
- moved R6 0.65 mm to (45.6, 89.0)
Routing:
- net GND: track 24.7 -> 23.8 mm, vias 17 -> 19
- net /LIPO STAT: track 15.6 -> 14.8 mm, vias 2 -> 0
- net +3V3: track 22.1 -> 21.4 mm
- net Net-(U1-PROG): track 2.20 -> 1.54 mm
- net /LED1: track 16.4 -> 16.9 mm
Other:
- board text added: "Rev01"

Commit message: Improve led footprint
Parts:
- D1, D2, D3, D4, D5, D6: footprint LTST-C230KRKT:LED_LTST-C230KRKT -> LTST-C230KRKT:Custom LTST-C230KRKT
- moved R5 5.66 mm to (62.0, 77.0), turned to -90 degrees
- moved R7 5.66 mm to (42.0, 77.0), turned to 90 degrees
- moved R1 5.03 mm to (46.5, 76.5), turned to 0 degrees
- moved R2 5.03 mm to (50.5, 76.5), turned to 0 degrees
- moved R3 5.03 mm to (54.5, 76.5), turned to 0 degrees
- moved R4 5.03 mm to (58.5, 76.5), turned to 0 degrees
Connections:
- R1 pad 1: +3V3 -> Net-(D1-K)
- R1 pad 2: Net-(D1-PadA) -> /LED1
- R2 pad 1: +3V3 -> Net-(D2-K)
- R2 pad 2: Net-(D2-PadA) -> /LED2
- R3 pad 1: +3V3 -> Net-(D3-K)
- R3 pad 2: Net-(D3-PadA) -> /LED3
- R4 pad 1: +3V3 -> Net-(D4-K)
- R4 pad 2: Net-(D4-PadA) -> /LED4
- R5 pad 1: +3V3 -> Net-(D5-K)
- R5 pad 2: Net-(D5-PadA) -> /LED5
- R7 pad 1: Net-(D6-PadA) -> /LIPO STAT
- R7 pad 2: +VBUS -> Net-(D6-K)
Routing:
- net +3V3: track 21.4 -> 17.5 mm
- net /LED5: track 7.41 -> 4.68 mm
- net +VBUS: track 29.3 -> 31.9 mm
- net /LED3: track 10.1 -> 7.59 mm
- net /LED4: track 7.64 -> 5.51 mm
- net /LED2: track 13.5 -> 11.4 mm
- net /LIPO STAT: track 14.8 -> 12.7 mm
- net Net-(D6-PadA): track 2.00 -> 0.00 mm
- net Net-(D3-PadA): track 1.98 -> 0.00 mm
- net Net-(D2-PadA): track 1.98 -> 0.00 mm
- net Net-(D5-PadA): track 1.98 -> 0.00 mm
- net Net-(D4-PadA): track 1.98 -> 0.00 mm
- net Net-(D1-PadA): track 1.98 -> 0.00 mm
- net /LED1: track 16.9 -> 15.0 mm
- net Net-(D4-K): track 0.00 -> 1.60 mm
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